File: IR-Sensor.sch (KiCad schematic (older format))
At the start: 20 parts, among them P1 CONN_01X04, Q1 2N7002, U1 TSSP77038, U2 MIC1557

Commit message: PCB empezada
Parts:
- Q1: footprint TO_SOT_Packages_SMD:SOT-23 -> TO_SOT_Packages_SMD:SOT-323_SC-70
Changed lines of the file:
@@
 F 0 "Q1" H 8005 3946 50  0000 L CNN
 F 1 "2N7002" H 8005 3855 50  0000 L CNN
-F 2 "TO_SOT_Packages_SMD:SOT-23" H 8000 3825 50  0001 L CIN
+F 2 "TO_SOT_Packages_SMD:SOT-323_SC-70" H 8000 3825 50  0001 L CIN
 F 3 "https://www.fairchildsemi.com/datasheets/2N/2N7002.pdf" H 7800 3900 50  0001 L CNN
 	1    7800 3900
